Commit message: file path fixes

File: urdf/custom.urdf (robot description, URDF)
Before this commit: robot None, 1 links, 1 joints
Links:
- added link sensor_offset, mass 0.01; visual box size=0.05 0.05 0.05
Joints:
- removed joint rad_joint
- added joint radiation_sensor_joint: type fixed, parent sensor_offset, child radiation_sensor, origin xyz=0 0 0 rpy=0 0 0
- added joint sensor_joint: type fixed, parent chassis_link, child sensor_offset, origin xyz=0 0 0 rpy=0 0 0

Commit message: Fixed issue with sensor offset

File: urdf/custom.urdf (robot description, URDF)
Before this commit: robot None, 2 links, 2 joints
Links:
- removed link sensor_offset
- link radiation_sensor: mass 0.01 -> 0.001
Joints:
- removed joint radiation_sensor_joint
- removed joint sensor_joint
- added joint radiation_sensor: type fixed, parent chassis_link, child radiation_sensor, origin xyz=0 0 1 rpy=0 0 0

Commit message: Fixed issue with sensor offset

File: urdf/custom.urdf (robot description, URDF)
Before this commit: robot None, 1 links, 1 joints
Links:
- link radiation_sensor: mass 0.01 -> 0.001
Joints:
- removed joint rad_joint
- added joint radiation_sensor: type fixed, parent chassis_link, child radiation_sensor, origin xyz=0 0 1 rpy=0 0 0

Commit message: update

File: urdf/custom.urdf (robot description, URDF)
Before this commit: robot None, 1 links, 1 joints
Joints:
- joint radiation_sensor: origin xyz=0 0 1 rpy=0 0 0 -> xyz=0 0 0 rpy=0 0 0
